File: 4 key with encoder.brd (EAGLE design)
At the start: 98.1 x 42.9 mm, 24 parts, among them SW1 KEYSWITCH-PLAIN-MXHS-1U, SW2 KEYSWITCH-PLAIN-MXHS-1U, SW3 KEYSWITCH-PLAIN-MXHS-1U, SW4 KEYSWITCH-PLAIN-MXHS-1U, SW5 KEYSWITCH-PLAIN-MXHS-1U, SW6 KEYSWITCH-PLAIN-MXHS-1U

Commit message: updates to board
Routing:
- net N$17: track 26.0 -> 26.9 mm
Other:
- board size 98.1 x 42.9 mm -> 105.2 x 42.9 mm
Changed lines of the file:
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@@
 <drawing>
 <settings>
-<setting alwaysvectorfont="yes"/>
+<setting alwaysvectorfont="no"/>
 <setting verticaltext="up"/>
 </settings>
@@
 <board>
 <plain>
-<wire x1="0" y1="0" x2="98.0875" y2="0" width="0" layer="20"/>
-<wire x1="98.0875" y1="0" x2="98.0875" y2="42.85" width="0" layer="20"/>
-<wire x1="98.0875" y1="42.85" x2="0" y2="42.85" width="0" layer="20"/>
-<wire x1="0" y1="42.85" x2="0" y2="0" width="0" layer="20"/>
+<wire x1="0" y1="24.85" x2="0" y2="18" width="0" layer="20"/>
+<wire x1="0" y1="18" x2="18" y2="0" width="0" layer="20" curve="90"/>
+<wire x1="18" y1="0" x2="100.23125" y2="0" width="0" layer="20"/>
+<wire x1="100.23125" y1="0" x2="105.23125" y2="5" width="0" layer="20" curve="90"/>
+<wire x1="105.23125" y1="5" x2="105.23125" y2="37.85" width="0" layer="20"/>
+<wire x1="105.23125" y1="37.85" x2="100.23125" y2="42.85" width="0" layer="20" curve="90"/>
+<wire x1="100.23125" y1="42.85" x2="18" y2="42.85" width="0" layer="20"/>
+<wire x1="18" y1="42.85" x2="0" y2="24.85" width="0" layer="20" curve="90"/>
 <circle x="19.05" y="21.43125" radius="21.298546875" width="0.1524" layer="51"/>
+<circle x="8.334375" y="34.528125" radius="3" width="0.1" layer="20"/>
+<circle x="8.334375" y="8.334375" radius="3" width="0.1" layer="20"/>
+<circle x="100.0125" y="38.1" radius="3" width="0.1" layer="20"/>
+<circle x="100.0125" y="4.7625" radius="3" width="0.1" layer="20"/>
 </plain>
 <attributes>
@@
 <contactref element="LED9" pad="4-DIN"/>
 <wire x1="6.5" y1="19" x2="5.5" y2="19" width="0.1524" layer="16"/>
-<wire x1="10" y1="22.5" x2="6.5" y2="19" width="0.1524" layer="1"/>
-<wire x1="10" y1="31" x2="10" y2="22.5" width="0.1524" layer="1"/>
-<wire x1="17" y1="38" x2="10" y2="31" width="0.1524" layer="16"/>
-<wire x1="18" y1="38" x2="17" y2="38" width="0.1524" layer="16"/>
+<wire x1="8.809375" y1="21.309375" x2="6.5" y2="19" width="0.1524" layer="1"/>
+<wire x1="10" y1="31" x2="8.809375" y2="29.809375" width="0.1524" layer="1"/>
+<wire x1="8.809375" y1="29.809375" x2="8.809375" y2="21.309375" width="0.1524" layer="1"/>
+<wire x1="18.3" y1="38.36875" x2="18.3" y2="36.91875" width="0.1524" layer="16"/>
+<wire x1="18.3" y1="36.91875" x2="12.38125" y2="31" width="0.1524" layer="16"/>
+<wire x1="12.38125" y1="31" x2="10" y2="31" width="0.1524" layer="16"/>
 <wire x1="5.5" y1="19" x2="5.5125" y2="18.78125" width="0.1524" layer="16"/>
-<wire x1="18" y1="38" x2="18.3" y2="38.36875" width="0.1524" layer="16"/>
 <via x="6.5" y="19" extent="1-16" drill="0.35"/>
 <via x="10" y="31" extent="1-16" drill="0.35"/>

Commit message: updates to board
Routing:
- net N$16: track 50.3 -> 43.9 mm
Changed lines of the file:
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@@
 <wire x1="11" y1="17" x2="18" y2="10" width="0.1524" layer="16"/>
 <wire x1="4" y1="17" x2="11" y2="17" width="0.1524" layer="16"/>
-<wire x1="2.5" y1="18.5" x2="4" y2="17" width="0.1524" layer="16"/>
-<wire x1="2.5" y1="30" x2="2.5" y2="18.5" width="0.1524" layer="16"/>
-<wire x1="18" y1="30" x2="2.5" y2="30" width="0.1524" layer="16"/>
+<wire x1="18" y1="30" x2="9.384775" y2="30" width="0.1524" layer="16"/>
+<wire x1="9.384775" y1="30" x2="4" y2="17" width="0.1524" layer="16" curve="135"/>
 <wire x1="19.5" y1="31.5" x2="18" y2="30" width="0.1524" layer="16"/>
 <wire x1="19.5" y1="33" x2="19.5" y2="31.5" width="0.1524" layer="16"/>

Commit message: tweaks
Parts:
- added S1: (no value), keeb-library:B3F-10XX
- B1: value SPARKFUN_PRO_MICRO -> (none)
- D1, D2, D3, D4, D5, D6: device keeb-library:DIODE_HAND -> keeb-library:SOD-123
- moved D6 2.66 mm to (44.1, 9.52), flipped to the bottom
- moved D5 2.66 mm to (44.1, 28.6), flipped to the bottom
- moved D3 2.66 mm to (63.1, 9.52), flipped to the bottom
- moved D1 2.66 mm to (63.1, 28.6), flipped to the bottom
- moved D4 2.66 mm to (82.2, 9.52), flipped to the bottom
- moved D2 2.66 mm to (82.2, 28.6), flipped to the bottom
- moved LED2 0.60 mm to (69.0, 25.6)
- moved LED5 0.60 mm to (69.0, 6.54)
- moved LED1 0.60 mm to (50.0, 25.6)
- moved LED4 0.60 mm to (50.0, 6.54)
- moved LED3 0.60 mm to (88.1, 25.6)
- moved LED6 0.60 mm to (88.1, 6.54)
Connections:
- new net RESET: B1.22, S1.1, S1.2
- net COL0: now also D5.C, D6.C; no longer D5.C1, D5.C2, D5.C3, D6.C1, D6.C2, D6.C3
- net COL1: now also D1.C, D3.C; no longer D1.C1, D1.C2, D1.C3, D3.C1, D3.C2, D3.C3
- net COL2: now also D2.C, D4.C; no longer D2.C1, D2.C2, D2.C3, D4.C1, D4.C2, D4.C3
- net GND: now also S1.3, S1.4
- net N$1: now also D5.A; no longer D5.A1, D5.A2, D5.A3
- net N$2: now also D6.A; no longer D6.A1, D6.A2, D6.A3
- net N$3: now also D3.A; no longer D3.A1, D3.A2, D3.A3
- net N$4: now also D1.A; no longer D1.A1, D1.A2, D1.A3
- net N$5: now also D2.A; no longer D2.A1, D2.A2, D2.A3
- net N$6: now also D4.A; no longer D4.A1, D4.A2, D4.A3
Routing:
- net GND: track 257.0 -> 0.00 mm, vias 6 -> 0
- net 5.0V: track 215.3 -> 0.00 mm
- net N$15: track 78.0 -> 0.00 mm
- net COL2: track 77.8 -> 0.00 mm
- net ROW1: track 77.5 -> 0.00 mm, vias 1 -> 0
- net N$12: track 77.0 -> 0.00 mm, vias 2 -> 0
- net ROW0: track 77.0 -> 0.00 mm, vias 1 -> 0
- net COL1: track 64.9 -> 0.00 mm
- net N$16: track 43.9 -> 0.00 mm
- net N$18: track 41.1 -> 0.00 mm, vias 2 -> 0
- net LED: track 34.3 -> 0.00 mm, vias 1 -> 0
- net COL0: track 29.0 -> 0.00 mm
- net N$17: track 26.9 -> 0.00 mm, vias 2 -> 0
- net N$11: track 14.4 -> 0.00 mm
- net N$8: track 14.4 -> 0.00 mm
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Other:
- board size 105.2 x 42.9 mm -> 96.4 x 40.5 mm
