File: 4 key with encoder.sch (EAGLE design)
At the start: 24 parts, among them SW1 KEYSWITCH-PLAIN-MXHS-1U, SW2 KEYSWITCH-PLAIN-MXHS-1U, SW3 KEYSWITCH-PLAIN-MXHS-1U, SW4 KEYSWITCH-PLAIN-MXHS-1U, SW5 KEYSWITCH-PLAIN-MXHS-1U, SW6 KEYSWITCH-PLAIN-MXHS-1U

Commit message: tweaks
Parts:
- added S1: (no value), keeb-library:10-XX
- B1: value SPARKFUN_PRO_MICRO -> (none)
- D1, D2, D3, D4, D5, D6: device keeb-library:DIODE-HAND -> keeb-library:DIODE-SOD-123
Connections:
- new net RESET: B1.RESET, S1.S, S1.S1
- net GND: now also S1.P, S1.P1
