File: 6 key with encoder.sch (EAGLE design)
At the start: 25 parts, among them SW1 KEYSWITCH-PLAIN-MXHS-1U, SW2 KEYSWITCH-PLAIN-MXHS-1U, SW3 KEYSWITCH-PLAIN-MXHS-1U, SW4 KEYSWITCH-PLAIN-MXHS-1U, SW5 KEYSWITCH-PLAIN-MXHS-1U, SW6 KEYSWITCH-PLAIN-MXHS-1U

Commit message: production 12-6-2021
Parts:
- added D7: (no value), keeb-library:DIODE-SOD-123
Connections:
- removed net N$24: ROTENC.P$A
- removed net N$25: ROTENC.P$B
- removed net N$26: ROTENC.P$1
- new net ENC_A: B1.A0, ROTENC.P$A
- new net ENC_B: B1.A2, ROTENC.P$B
- new net N$7: D7.A, ROTENC.P$2
- new net ROW2: B1.A1, ROTENC.P$1
- net COL2: now also D7.C
- net GND: no longer ROTENC.P$2
